File: kicad/esp32-pc-control/esp32-pc-control.kicad_sch (KiCad schematic)
At the start: 11 parts, among them U1 PC817, U2 PC817, U3 PC817

Commit message: Translate build guide to English and simplify assembly notes
Other:
- note added: "Power Supply (optional when powered through USB-C)"
- note added: "RESET (GPIO26) (optional; POWER can be used to turn the PC off and on again)"
- note added: "Status input from PWR_LED"
- note removed: "Power Supply (not required when the USB-C port is used for power delivery)"
- note removed: "RESET (GPIO26) (not required, as you can use the power switch for a hard reset.)"
- note removed: "Status imput from PWR_LED"
Changed lines of the file:
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@@
 		)
 	)
-	(text "Status imput from PWR_LED"
+	(text "Status input from PWR_LED"
 		(exclude_from_sim no)
 		(at 107.95 146.812 0)
@@
 		)
 	)
-	(text "Power Supply\n(not required when the USB-C port is used for power delivery)"
+	(text "Power Supply\n(optional when powered through USB-C)"
 		(exclude_from_sim no)
 		(at 164.084 37.592 0)
@@
 		)
 	)
-	(text "RESET (GPIO26)\n(not required, as you can use the power switch for a hard reset.)"
+	(text "RESET (GPIO26)\n(optional; POWER can be used to turn the PC off and on again)"
 		(exclude_from_sim no)
 		(at 163.576 104.902 0)
